File: alu_xor_2bits.brd (EAGLE design)
At the start: 116.8 x 97.5 mm, 66 parts, among them IC1 74LS86N, IC10 74LS86N, IC15 74ALS00N, IC18 74LS151N, IC2 74ALS00N, IC3 74LS151N, IC4 74LS86N, IC5 74ALS00N, IC6 74LS151N, IC7 74LS86N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

Commit message: add functionality check
Connections:
- net N$2 renamed ADD0
- net N$24 renamed ADD1
- net N$33 renamed ADD2
- net N$38 renamed ADD3
Changed lines of the file:
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@@
 <via x="33.02" y="44.45" extent="1-16" drill="0.21"/>
 </signal>
-<signal name="N$2">
+<signal name="ADD0">
 <contactref element="IC1" pad="8"/>
 <contactref element="IC18" pad="2"/>
@@
 <wire x1="-5.08" y1="-17.78" x2="-5.08" y2="-30.48" width="0" layer="19" extent="1-1"/>
 </signal>
-<signal name="N$24">
+<signal name="ADD1">
 <contactref element="IC4" pad="8"/>
 <contactref element="IC3" pad="2"/>
@@
 <wire x1="-5.08" y1="-55.88" x2="-5.08" y2="-81.28" width="0" layer="19" extent="1-1"/>
 </signal>
-<signal name="N$33">
+<signal name="ADD2">
 <contactref element="IC7" pad="8"/>
 <contactref element="IC6" pad="2"/>
@@
 <wire x1="-5.08" y1="-68.58" x2="-5.08" y2="-106.68" width="0" layer="19" extent="1-1"/>
 </signal>
-<signal name="N$38">
+<signal name="ADD3">
 <contactref element="IC10" pad="8"/>
 <contactref element="IC9" pad="2"/>
