File: alu_xor_2bits.sch (EAGLE design)
At the start: 66 parts, among them IC1 74LS86N, IC10 74LS86N, IC15 74ALS00N, IC18 74LS151N, IC2 74ALS00N, IC3 74LS151N, IC4 74LS86N, IC5 74ALS00N, IC6 74LS151N, IC7 74LS86N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

Commit message: add functionality check
Connections:
- net N$2 renamed ADD0
- net N$24 renamed ADD1
- net N$33 renamed ADD2
- net N$38 renamed ADD3
Changed lines of the file:
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@@
 </segment>
 </net>
-<net name="N$2" class="0">
+<net name="ADD0" class="0">
 <segment>
 <pinref part="IC1" gate="C" pin="O"/>
 <wire x1="73.66" y1="137.16" x2="73.66" y2="68.58" width="0.1524" layer="91"/>
 <pinref part="IC18" gate="A" pin="D2"/>
+<label x="73.66" y="86.36" size="1.778" layer="95" rot="R90"/>
 </segment>
 </net>
@@
 </segment>
 </net>
-<net name="N$24" class="0">
+<net name="ADD1" class="0">
 <segment>
 <pinref part="IC4" gate="C" pin="O"/>
 <wire x1="137.16" y1="137.16" x2="137.16" y2="68.58" width="0.1524" layer="91"/>
 <pinref part="IC3" gate="A" pin="D2"/>
+<label x="137.16" y="86.36" size="1.778" layer="95" rot="R90"/>
 </segment>
 </net>
@@
 </segment>
 </net>
-<net name="N$33" class="0">
+<net name="ADD2" class="0">
 <segment>
 <pinref part="IC7" gate="C" pin="O"/>
 <wire x1="200.66" y1="137.16" x2="200.66" y2="68.58" width="0.1524" layer="91"/>
 <pinref part="IC6" gate="A" pin="D2"/>
+<label x="200.66" y="88.9" size="1.778" layer="95" rot="R90"/>
 </segment>
 </net>
@@
 </segment>
 </net>
-<net name="N$38" class="0">
+<net name="ADD3" class="0">
 <segment>
 <pinref part="IC10" gate="C" pin="O"/>
 <wire x1="264.16" y1="137.16" x2="264.16" y2="68.58" width="0.1524" layer="91"/>
 <pinref part="IC9" gate="A" pin="D2"/>
-</segment>
-</net>
+<label x="264.16" y="86.36" size="1.778" layer="95" rot="R90"/>
+</segment>
+</net>
